File: KICAD/sourcebox/sourcebox.sch (KiCad schematic (older format))
At the start: 21 parts, among them J1 Conn_02x15_Odd_Even, U1 74LS76, U10 74LS76, U11 74LS10, U12 74LS02, U13 74LS86, U14 74LS125, U2 74LS393, U3 74LS393, U4 74LS30, U5 74LS74, U6 74LS00, U7 74LS04, U9 74LS02

Commit message: [KICAD] a lot of work on the source box schematics
Parts:
- removed J1: Conn_02x15_Odd_Even, symbol Connector:Conn_02x15_Odd_Even
- added J1: Conn_02x16_Counter_Clockwise, symbol Connector:Conn_02x16_Counter_Clockwise
- added J2: JAMMA_CONNECTOR, symbol jamma_connector:JAMMA_CONNECTOR
- added J3, J4: Conn_02x05_Counter_Clockwise, symbol Connector:Conn_02x05_Counter_Clockwise
- added J5: Conn_02x04_Counter_Clockwise, symbol Connector:Conn_02x04_Counter_Clockwise
- added J6: Conn_01x02, symbol Connector:Conn_01x02
- added JP1, JP2, JP3: Jumper, symbol device:Jumper
- added R10, R11, R12, R13, R14, R15, R16, R17, R18, R19, R20, R21, R22, R5, R6, R7, R8, R9: 2.2K, symbol device:R
Connections:
- net labels added: +12V, -ACTIVE_GAME_VIDEO, -CSYNC, -HSYNC, -P1_BUTTON_1, -P1_BUTTON_2, -P1_BUTTON_3, -P1_COIN, -P1_DOWN, -P1_LEFT, -P1_RIGHT, -P1_START, -P1_UP, -P2_BUTTON_1, -P2_BUTTON_2, -P2_BUTTON_3, -P2_COIN, -P2_DOWN, -P2_LEFT, -P2_RIGHT, -P2_START, -P2_UP, -VDC, BLANK, GAME_VIDEO_B, GAME_VIDEO_G, GAME_VIDEO_R
- net labels removed: GAME_VIDEO, HSYNC
- wire segments 255 -> 434
- no-connect marks 3 -> 12
Other:
- note added: "A generic board for prototyping\ncustom discrete TV/Arcade games\n"
- note added: "BOARD CONNECTORS"
- note added: "COMPOSITE VIDEO OUT"
- note added: "GAME MODULE INTERFACE"
- note added: "HORIZONTAL BEAM POSITION"
- note added: "JAMMA INTERFACE"
- note added: "MONOCHROME COMPOSITE VIDEO"
- note added: "PIXEL CLOCK SOURCE"
- note added: "PLAYER #1 INPUTS"
- note added: "PLAYER #2 INPUTS"
- note added: "POWER CONNECTOR"
- note added: "SOURCEBOX"
- note added: "STANDARD TV SIGNALING"
- note added: "SYNC, RESET & BLANK SIGNALS"
- note added: "VERTICAL BEAM POSITION"

Commit message: [KICAD] SourceBox test-pattern generator and additional tweaks in the design
Parts:
- removed unit 4 of U12
- removed unit 4 of U9
- removed unit 2 of U9
- removed unit 1 of U9
- added JP4, JP5, JP6: Jumper, symbol device:Jumper
- added unit 3 of U11
- added unit 3 of U13
- added unit 4 of U13
- added U15: 74LS08, symbol Logic_74xx:74LS08
- added unit 5 of U7
- added unit 4 of U7
Connections:
- net labels added: -BLANK, ACTIVE_BLUE, ACTIVE_GREEN, ACTIVE_MONOCHROME_VIDEO, ACTIVE_RED
- net labels removed: -ACTIVE_GAME_VIDEO, BLANK
- wire segments 434 -> 447
Other:
- note added: "16x16 Red checkerboard\n\n\n\n32x32 Green checkerboard\n\n\n\n8x8 Blue windows\n(only visible when\n player #1 start\n button is pressed)"
- note added: "RESTRICT RGB SIGNALS\nTO BE ACTIVE ONLY\nWHEN OUTSIDE OF\nBLANKING INTERVALS"
- note added: "SAMPLE VIDEO GENERATOR"
- note added: "Use this in order to test the board."

Commit message: [KICAD] Adding audio circuits
Parts:
- added C2: 100uF, symbol device:CP1
- added C3, C4: 10uF, symbol device:CP1
- added J7: Conn_01x02, symbol Connector:Conn_01x02
- added JP7: Jumper, symbol device:Jumper
- added R23: 330R, symbol device:R
- added R24: 2.2k, symbol device:R
- added RV1: 50K, symbol device:POT
- added U8: LM386, symbol audio:LM386
- added unit 1 of U9
- added unit 4 of U9
- added unit 2 of U9
Connections:
- net labels added: AUDIO_OUT, GAME_AUDIO
- wire segments 447 -> 487
- no-connect marks 12 -> 10
Other:
- note added: "493Hz tone when\nholding P1 DOWN"
- note added: "987Hz tone when\nholding P1 UP"
- note added: "AMP AUDIO OUT"
- note added: "AUDIO AMPLIFIER"
- note added: "SAMPLE AUDIO & VIDEO GENERATION"
- note removed: "SAMPLE VIDEO GENERATOR"

Commit message: [KICAD] Adding VGA-OUT connector
Parts:
- added J8: DB15_Female_HighDensity, symbol Connector:DB15_Female_HighDensity
Connections:
- net labels added: VSYNC
- wire segments 487 -> 505
- no-connect marks 10 -> 15
Other:
- note added: "VGA OUTPUT"

Commit message: [KICAD] draw sync/blank diagrams and annotate flip-flops
Other:
- note added: "-HSYNC"
- note added: "-R/-S\nFLIP-FLOP"
- note added: "-RESET\n"
- note added: "-SET\n"
- note added: "-VSYNC"
- note added: "0"
- note added: "16"
- note added: "32"
- note added: "4"
- note added: "64"
- note added: "8"
- note added: "80"
- note added: "H-COUNT"
- note added: "HBLANK"
- note added: "R/S\nFLIP-FLOP"
- note added: "RESET"
- note added: "SET"
- note added: "V-COUNT"
- note added: "VBLANK"
- note added: "VIDEO RESOLUTION: 375x246\n\nTOTAL-H: 455\nTOTAL-V: 262\nHBLANK: 80\nVBLANK: 16"

Commit message: [KICAD] Fix Vsync circuit
Parts:
- removed J1: Conn_02x16_Counter_Clockwise, symbol Connector:Conn_02x16_Counter_Clockwise
- added J1: Conn_02x18_Counter_Clockwise, symbol Connector:Conn_02x18_Counter_Clockwise
Connections:
- net labels added: -VSYNC
- net labels removed: VSYNC
- wire segments 505 -> 509
